Commit message: third commit

File: kitchen_gazebo/robots/kitchen_gazebo.URDF (robot description, URDF)
Before this commit: robot kitchen_gazebo, 6 links, 5 joints
Links:
- link base_link: mass 24756.9002576438 -> 24691.7377583292
- link drawer_left: mass 9.47751493301134 -> 9.47751493301151
- link water_pipe: mass 0.278769423544699 -> 0.278769423544692
Joints:
- joint drawer_left: limit lower=0 upper=0.55 effort=1000.0 velocity=0.275 -> lower=0 upper=0.55 effort=1000.0 velocity=0.5
- joint drawer_right: limit lower=0 upper=0.55 effort=1000.0 velocity=0.275 -> lower=0 upper=0.55 effort=1000.0 velocity=0.5
